Commit message: feat: publish verified single-camera and TCP planning model
Preserve calibrated-model support from fe0c98d and integrate camera/TCP frames, current gripper mounting and shared position limits. The six files match the isolated validated candidate; generated model elements are unchanged. Validation covers offline/mock PLAN-ONLY diagnostics, not physical grasp execution.

File: urdf/aubo_i5.urdf.xacro (robot description, xacro)
@@ -1,4 +1,5 @@
 <?xml version="1.0"?>
 <robot name="aubo_i5" xmlns:xacro="http://wiki.ros.org/xacro">
+  <xacro:include filename="$(find aubo_joint_limits)/config/position_limits.xacro"/>
   <dh_type type="modified"/>
   <safety_para singularity_consistent="0.02 0.01 10 0.2 0.045 10"/>
@@ -53,5 +54,5 @@
     <child link="shoulder_Link" />
     <axis xyz="0 0 1" />
-    <limit lower="-6.283185307179586476925286766559" upper="6.283185307179586476925286766559" effort="133" start_stop="207" velocity="2.5964" />
+    <limit lower="${arm_position_limits['shoulder_joint']['lower']}" upper="${arm_position_limits['shoulder_joint']['upper']}" effort="133" start_stop="207" velocity="2.5964" />
   </joint>
   <link name="upperArm_Link">
@@ -82,5 +83,5 @@
     <child link="upperArm_Link" />
     <axis xyz="0 0 1" />
-    <limit lower="-6.283185307179586476925286766559" upper="6.283185307179586476925286766559" effort="133" start_stop="207" velocity="2.5964" />
+    <limit lower="${arm_position_limits['upperArm_joint']['lower']}" upper="${arm_position_limits['upperArm_joint']['upper']}" effort="133" start_stop="207" velocity="2.5964" />
   </joint>
   <link name="foreArm_Link">
@@ -111,5 +112,5 @@
     <child link="foreArm_Link" />
     <axis xyz="0 0 1" />
-    <limit lower="-6.283185307179586476925286766559" upper="6.283185307179586476925286766559" effort="133" start_stop="207" velocity="2.5964" />
+    <limit lower="${arm_position_limits['foreArm_joint']['lower']}" upper="${arm_position_limits['foreArm_joint']['upper']}" effort="133" start_stop="207" velocity="2.5964" />
   </joint>
   <link name="wrist1_Link">
@@ -140,5 +141,5 @@
     <child link="wrist1_Link" />
     <axis xyz="0 0 1" />
-    <limit lower="-6.283185307179586476925286766559" upper="6.283185307179586476925286766559" effort="13.5" start_stop="34" velocity="3.1105" />
+    <limit lower="${arm_position_limits['wrist1_joint']['lower']}" upper="${arm_position_limits['wrist1_joint']['upper']}" effort="13.5" start_stop="34" velocity="3.1105" />
   </joint>
   <link name="wrist2_Link">
@@ -169,5 +170,5 @@
     <child link="wrist2_Link" />
     <axis xyz="0 0 1" />
-    <limit lower="-6.283185307179586476925286766559" upper="6.283185307179586476925286766559" effort="13.5" start_stop="34" velocity="3.1105" />
+    <limit lower="${arm_position_limits['wrist2_joint']['lower']}" upper="${arm_position_limits['wrist2_joint']['upper']}" effort="13.5" start_stop="34" velocity="3.1105" />
   </joint>
   <link name="wrist3_Link">
@@ -198,5 +199,5 @@
     <child link="wrist3_Link" />
     <axis xyz="0 0 1" />
-    <limit lower="-6.283185307179586476925286766559" upper="6.283185307179586476925286766559" effort="13.5" start_stop="34" velocity="3.1105" />
+    <limit lower="${arm_position_limits['wrist3_joint']['lower']}" upper="${arm_position_limits['wrist3_joint']['upper']}" effort="13.5" start_stop="34" velocity="3.1105" />
   </joint>
   <link name="world" />

File: urdf/xacro/inc/aubo.ros2_control.xacro (robot description, xacro)
@@ -1,5 +1,7 @@
 <?xml version="1.0"?>
 <robot xmlns:xacro="http://www.ros.org/wiki/xacro">
-  <xacro:macro name="aubo_ros2_control" params="name prefix use_fake_hardware:=false robot_ip">
+  <xacro:macro name="aubo_ros2_control" params="name prefix use_fake_hardware:=false robot_ip position_limits:=${dict()}">
+    <xacro:property name="legacy_min" value="{-2*pi}"/>
+    <xacro:property name="legacy_max" value="{2*pi}"/>
     <ros2_control name="${name}" type="system">
        <hardware>
@@ -16,6 +18,6 @@
       <joint name="shoulder_joint">
         <command_interface name="position">
-          <param name="min">{-2*pi}</param>
-          <param name="max">{2*pi}</param>
+          <param name="min">${position_limits['shoulder_joint']['lower'] if position_limits else legacy_min}</param>
+          <param name="max">${position_limits['shoulder_joint']['upper'] if position_limits else legacy_max}</param>
         </command_interface>
         <command_interface name="velocity"/>
@@ -27,6 +29,6 @@
       <joint name="upperArm_joint">
         <command_interface name="position">
-          <param name="min">{-2*pi}</param>
-          <param name="max">{2*pi}</param>
+          <param name="min">${position_limits['upperArm_joint']['lower'] if position_limits else legacy_min}</param>
+          <param name="max">${position_limits['upperArm_joint']['upper'] if position_limits else legacy_max}</param>
         </command_interface>
         <command_interface name="velocity"/>
@@ -38,6 +40,6 @@
       <joint name="foreArm_joint">
         <command_interface name="position">
-          <param name="min">-2.41</param>
-          <param name="max">2.41</param>
+          <param name="min">${position_limits['foreArm_joint']['lower'] if position_limits else -2.41}</param>
+          <param name="max">${position_limits['foreArm_joint']['upper'] if position_limits else 2.41}</param>
         </command_interface>
         <command_interface name="velocity"/>
@@ -49,6 +51,6 @@
       <joint name="wrist1_joint">
         <command_interface name="position">
-          <param name="min">-2.66</param>
-          <param name="max">2.66</param>
+          <param name="min">${position_limits['wrist1_joint']['lower'] if position_limits else -2.66}</param>
+          <param name="max">${position_limits['wrist1_joint']['upper'] if position_limits else 2.66}</param>
         </command_interface>
         <command_interface name="velocity"/>
@@ -60,6 +62,6 @@
       <joint name="wrist2_joint">
         <command_interface name="position">
-          <param name="min">{-2*pi}</param>
-          <param name="max">{2*pi}</param>
+          <param name="min">${position_limits['wrist2_joint']['lower'] if position_limits else legacy_min}</param>
+          <param name="max">${position_limits['wrist2_joint']['upper'] if position_limits else legacy_max}</param>
         </command_interface>
         <command_interface name="velocity"/>
@@ -71,6 +73,6 @@
       <joint name="wrist3_joint">
         <command_interface name="position">
-          <param name="min">-2.23</param>
-          <param name="max">2.23</param>
+          <param name="min">${position_limits['wrist3_joint']['lower'] if position_limits else -2.23}</param>
+          <param name="max">${position_limits['wrist3_joint']['upper'] if position_limits else 2.23}</param>
         </command_interface>
         <command_interface name="velocity"/>

File: urdf/xacro/inc/aubo_ros2.xacro (robot description, xacro)
@@ -19,4 +19,7 @@
   </xacro:if>
   <xacro:include filename="$(find aubo_description)/urdf/xacro/inc/aubo_ros2_macro.xacro"/>
+  <xacro:if value="${aubo_type == 'aubo_i5'}">
+    <xacro:include filename="$(find aubo_joint_limits)/config/position_limits.xacro"/>
+  </xacro:if>
   <xacro:aubo_robot
     transmission_hw_interface="$(arg transmission_hw_interface)"
@@ -30,6 +33,13 @@
     parent="ee_link"
     include_ros2_control="false">
-    <origin xyz="0 0 0.01" rpy="0 0 0"/>
+    <origin xyz="0 0 0.01" rpy="0 0 1.57079632679"/>
   </xacro:robotiq_gripper>
+  <!-- Robotiq 2F-85 grasp TCP -->
+  <link name="gripper_tcp"/>
+  <joint name="gripper_tcp_joint" type="fixed">
+    <parent link="robotiq_85_base_link"/>
+    <child link="gripper_tcp"/>
+    <origin xyz="0 0 0.136" rpy="0 0 0"/>
+  </joint>
   <!-- ros2_control -->
   <xacro:include filename="$(find aubo_description)/urdf/xacro/inc/aubo.ros2_control.xacro" />
@@ -38,4 +48,5 @@
     prefix=""
     use_fake_hardware="${use_fake_hardware}"
+    position_limits="${arm_position_limits if aubo_type == 'aubo_i5' else dict()}"
     robot_ip="${robot_ip}"/>
   <!-- Gripper selection is independent of the arm hardware. -->

File: urdf/xacro/inc/aubo_ros2_macro.xacro (robot description, xacro)
@@ -9,5 +9,15 @@
     </joint>
     <!-- Virtual end-effector frame; physical flange geometry belongs to wrist3_Link. -->
-<link name="ee_link"/>
+    <link name="ee_link"/>
+    <!-- Intel RealSense D435i camera base frame -->
+    <link name="camera_link"/>
+    <!-- Eye-in-Hand hand-eye calibration result 19_NO18 + TSAI -->
+    <joint name="camera_fixed_joint" type="fixed">
+      <parent link="ee_link"/>
+      <child link="camera_link"/>
+      <origin
+        xyz="0.08054669 -0.02160629 -0.00483282"
+        rpy="-2.53460119 -1.55296946 -0.60200016"/>
+    </joint>
     <transmission name="shoulder_trans">
       <type>transmission_interface/SimpleTransmission</type>
